File: hardware/trace.kicad_pcb (KiCad board)
At the start: 2 copper layers, 310 x 79 mm, 63 parts, among them Q1 DMG1012T, U1 LP2985-1.8, U10 IRS2092S, U11 INA240A1PW, U12 74AHCV17APW, U13 XPT2046TS, U14 INA253, U15 ATmega8U2-A, U16 AD7606, U17 THAT6261, U18 STM32F072RBIx, U19 FU540-C000, U2 LM317_SOT-223, U20 INA181, U21 LTC6226xDC, U22 LTC2294xUP, U23 LTC6269xDD, U24 WM8731CLSEFL, U25 BQ25570, U26 IS31FL3733-TQ, U27 PCA9685PW, U28 SN74CB3Q3384APW, U29 AD630ARZ, U3 LM317L_SOT-89, U4 LTC6362xDD, U5 PAM8908, U6 CS4265, U7 iC-HTG, U8 SN65HVD255D, U9 74HC4024

Commit message: finished inches
Parts:
- moved U19 36.1 mm to (276.0, 124.7)
- moved C11 22.4 mm to (39.6, 139.6)
- moved C12 22.4 mm to (51.4, 139.1)
- moved C14 22.4 mm to (69.6, 136.9)
- moved C13 22.4 mm to (61.3, 137.8)
- moved C15 22.4 mm to (76.7, 136.3)
Other:
- board size 310 x 79 mm -> 310 x 35 mm
- board text added: "0"

Commit message: stuff
Parts:
- added C1: 0201, Capacitor_SMD:C_0201_0603Metric, F.Cu at (126.3, 95.1)
- added C16: 1206, Capacitor_SMD:C_1206_3216Metric, F.Cu at (111.5, 93.5)
- added C17: 1210, Capacitor_SMD:C_1210_3225Metric, F.Cu at (125.0, 86.5)
- added C18: 1808, Capacitor_SMD:C_1808_4520Metric, F.Cu at (119.9, 87.4)
- added C19: 1812, Capacitor_SMD:C_1812_4532Metric, F.Cu at (113.4, 86.9)
- added C2: 0402, Capacitor_SMD:C_0402_1005Metric, F.Cu at (124.0, 94.9)
- added C20: 1825, Capacitor_SMD:C_1825_4564Metric, F.Cu at (123.2, 79.7)
- added C21: 2220, Capacitor_SMD:C_2220_5750Metric, F.Cu at (114.6, 79.8)
- added C22: 2225, Capacitor_SMD:C_2225_5664Metric, F.Cu at (105.9, 79.3)
- added C23: 3640, Capacitor_SMD:C_3640_9110Metric, F.Cu at (104.2, 90.4)
- added C24: 3, Capacitor_SMD:CP_Elec_3x5.4, F.Cu at (131.2, 78.6)
- added C25: 7.5, Capacitor_THT:CP_Radial_D7.5mm_P2.50mm, F.Cu at (163.7, 80.7)
- added C3: 0504, Capacitor_SMD:C_0504_1310Metric, F.Cu at (121.3, 94.8)
- added C4: 0603, Capacitor_SMD:C_0603_1608Metric, F.Cu at (118.3, 94.3)
- added C5: 0805, Capacitor_SMD:C_0805_2012Metric, F.Cu at (115.1, 94.1)
- added E$50: , NMOS-SYMB, B.Cu at (170.4, 85.4)
- added E$51: , PMOS-SYMB, B.Cu at (178.8, 85.4)
- added E$53: , LED-GUIDE, B.Cu at (178.7, 92.2)
- added E$54: , NPN-SYMB, B.Cu at (162.7, 85.4)
- added E$59: , PNP-SYMB, B.Cu at (187.2, 85.4)
- added L10: 0603, Inductor_SMD:L_0603_1608Metric, F.Cu at (222.6, 79.5)
- added L11: 0805, Inductor_SMD:L_0805_2012Metric, F.Cu at (222.8, 81.7)
- added L12: 1206, Inductor_SMD:L_1206_3216Metric, F.Cu at (223.4, 87.8)
- added L13: 1806, Inductor_SMD:L_1806_4516Metric, F.Cu at (224.1, 95.1)
- added L14: 2010, Inductor_SMD:L_2010_5025Metric, F.Cu at (213.8, 79.9)
- added L8: 0201, Inductor_SMD:L_0201_0603Metric, F.Cu at (221.8, 76.1)
- added L9: 0402, Inductor_SMD:L_0402_1005Metric, F.Cu at (222.0, 77.6)
- added R10: 0508, Resistor_SMD:R_0508_1220Metric, F.Cu at (84.9, 79.3)
- added R11: 0612, Resistor_SMD:R_0612_1632Metric, F.Cu at (85.5, 84.2)
- added R12: 0815, Resistor_SMD:R_0815_2038Metric, F.Cu at (85.9, 90.0)
- added R13: 1020, Resistor_SMD:R_1020_2550Metric, F.Cu at (86.4, 93.9)
- added R14: 1218, Resistor_SMD:R_1218_3246Metric, F.Cu at (78.9, 82.8)
- added R15: 1225, Resistor_SMD:R_1225_3264Metric, F.Cu at (78.0, 78.0)
- added R16: 2816, Resistor_SMD:R_2816_7142Metric, F.Cu at (69.3, 86.8)
- C8: value 6 -> 6.3
- U10, U11, U12, U13, U14, U15, U16, U17, U18, U19, U21, U22, U23, U24, U25, U26, U27, U28, U29, U4, U5, U6, U7, U8, U9: moved to B.Cu
- moved U5 208.7 mm to (67.2, 91.3), turned to 180 degrees
- moved U25 206.5 mm to (74.1, 91.0), turned to 180 degrees
- moved U7 200.5 mm to (81.5, 90.7), turned to 180 degrees
- moved U22 181.7 mm to (70.2, 80.9), turned to 180 degrees
- moved U17 179.0 mm to (81.1, 79.9), turned to 180 degrees
- moved U16 162.6 mm to (110.0, 85.1), turned to 180 degrees
- moved U24 149.0 mm to (89.5, 90.3), turned to 180 degrees
- moved U6 147.6 mm to (90.0, 78.8), turned to 180 degrees
- moved U21 132.4 mm to (150.2, 93.5), turned to 180 degrees
- moved U23 129.4 mm to (150.2, 81.7), turned to 180 degrees
- moved U4 128.6 mm to (150.1, 87.9), turned to 180 degrees
- moved U2 125.7 mm to (241.3, 80.6)
- moved U3 123.0 mm to (249.4, 80.3)
- moved U26 122.7 mm to (123.5, 85.1), turned to 180 degrees
- moved U20 120.7 mm to (255.7, 80.6), turned to 90 degrees
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Routing:
- net (no net): track 0.00 -> 120.8 mm
Other:
- outline, holes or cut-outs redrawn
- board text added: "0.45"
- board text added: "0.51"
- board text added: "0.57"
- board text added: "0.64"
- board text added: "0.72"
- board text added: "0.81"
- board text added: "0.91"
- board text added: "0201"
- board text added: "0402"
- board text added: "0504"
- board text added: "0508"
- board text added: "0603"
- board text added: "0612"
- board text added: "0805"
- board text added: "0815"
- board text added: "1.02"
- board text added: "1.15"
- board text added: "1.29"
- board text added: "1.45"
- board text added: "1.62"
- board text added: "1.82"
- board text added: "10.4x10.4"
- board text added: "1020"
- board text added: "10P5"
- board text added: "10x10.5"
- board text added: "11"
- board text added: "12"
- board text added: "1206"
- board text added: "1210"
- board text added: "1218"
- board text added: "1225"
- board text added: "13"
- board text added: "14"
- board text added: "15"
- board text added: "16"
- board text added: "17"
- board text added: "18"
- board text added: "1806"
- board text added: "1808"
- board text added: "1812"
- board text added: "1825"
- board text added: "19"
- board text added: "2.05"
- board text added: "2.3"
- board text added: "2.59"
- board text added: "2.9"
- board text added: "2010"
- board text added: "21"
- board text added: "22"
- board text added: "2220"
- board text added: "2225"
- board text added: "23"
- board text added: "24"
- board text added: "25"
- board text added: "2512"
- board text added: "3.26"
- board text added: "3640"
- board text added: "3x5.4"
- board text added: "4020"
- board text added: "4P2"
- board text added: "4x5.3"
- board text added: "5P2"
- board text added: "5x5.7"
- board text added: "6.3P2.5"
- board text added: "6.3x5.9"
- board text added: "6.3x6.3"
- board text added: "7.3x7.3"
- board text added: "7.5P2.5"
- board text added: "8"
- board text added: "8P3.5"
- board text added: "8x10.5"
- board text added: "9"
- board text added: "@notaroomba"
- board text added: "AWG"
- board text added: "BGA-64"
- board text added: "Capacitors"
- board text added: "DFN"
- board text added: "DFN-10"
- board text added: "DFN-6"
- board text added: "DFN-8"
- board text added: "DIODE SMA"
- board text added: "DIODE SMB"
- board text added: "DIODE SMC"
- board text added: "DIODE SMF"
- board text added: "ELEC"
- board text added: "General"
- board text added: "Inductors"
- board text added: "LQFP-64"
- board text added: "MM"
- board text added: "QFN"
- board text added: "QFN-16"
- board text added: "QFN-20"
- board text added: "QFN-24"
- board text added: "QFN-28"
- board text added: "QFN-32"
- board text added: "QFN-48"
- board text added: "QFN-64"
- board text added: "QFP"
- board text added: "Resistors"
- board text added: "SMD"
- board text added: "SOD-123"
- board text added: "SOD-323"
- board text added: "SOIC"
- board text added: "SOIC-14"
- board text added: "SOIC-16"
- board text added: "SOIC-20"
- board text added: "SOIC-8"
- board text added: "SOT-223"
- board text added: "SOT-23-5"
- board text added: "SOT-23-6"
- board text added: "SOT-323"
- board text added: "SOT-523"
- board text added: "SOT-89"
- board text added: "THT"
- board text added: "TQFP-32"
- board text added: "TQFP-48"
- board text added: "TSSOP"
- board text added: "TSSOP-14"
- board text added: "TSSOP-16"
- board text added: "TSSOP-20"
- board text added: "TSSOP-24"
- board text added: "TSSOP-28"
- board text added: "TSSOP-8"
- board text added: "Trace"
