File: hardware/trace.kicad_pcb (KiCad board)
At the start: 2 copper layers, 310 x 35 mm, 100 parts, among them Q1 DMG1012T, U1 LP2985-1.8, U10 IRS2092S, U11 INA240A1PW, U12 74AHCV17APW, U13 XPT2046TS, U14 INA253, U15 ATmega8U2-A, U16 AD7606, U17 THAT6261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

Commit message: fix text
Other:
- board text added: "2816"
